File: KosmoVoltsMain/KosmoVoltsMain.kicad_pcb (KiCad board)
At the start: 2 copper layers, 126.5 x 44 mm, 20 parts, among them J3 OUT, U1 TL072

Commit message: Manufacturing Update
Changed lines of the file:
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@@
       (disableapertmacros false)
       (usegerberextensions false)
-      (usegerberattributes true)
-      (usegerberadvancedattributes true)
+      (usegerberattributes false)
+      (usegerberadvancedattributes false)
       (creategerberjobfile true)
       (svguseinch false)
@@
       (outputformat 1)
       (mirror false)
-      (drillshape 1)
+      (drillshape 0)
       (scaleselection 1)
-      (outputdirectory "")
+      (outputdirectory "Gerbers/")
     )
   )
@@
     (fp_line (start -3.18 -22.88) (end -3.18 4.1) (layer "B.Fab") (width 0.1))
     (fp_line (start -3.18 4.1) (end -2.18 5.1) (layer "B.Fab") (width 0.1))
-    (pad "1" thru_hole roundrect (at 0 0 270) (size 1.7 1.7) (drill 1) (layers *.Cu *.Mask) (roundrect_rratio 0.147059)
+    (pad "1" thru_hole roundrect (at 0 0 270) (size 1.7 1.7) (drill 1) (layers *.Cu *.Mask) (roundrect_rratio 0.1470588235)
       (net 2 "/GATE1") (pinfunction "Pin_1") (pintype "passive"))
     (pad "2" thru_hole circle (at 2.54 0 270) (size 1.7 1.7) (drill 1) (layers *.Cu *.Mask)
@@
     (property "Vendor" "Tayda")
     (attr through_hole)
-    (fp_text reference "R2" (at 3.556 0.508 90) (layer "B.SilkS")
+    (fp_text reference "R2" (at -1.92 -0.1 180) (layer "B.SilkS")
       (effects (font (size 0.75 0.75) (thickness 0.15)) (justify mirror))
     )
@@
     (property "Vendor" "Tayda")
     (attr through_hole)
-    (fp_text reference "R3" (at 3.556 0.508 90) (layer "B.SilkS")
+    (fp_text reference "R3" (at -1.82 0 180) (layer "B.SilkS")
       (effects (font (size 0.75 0.75) (thickness 0.15)) (justify mirror))
     )
@@
     (property "Vendor" "Tayda")
     (attr through_hole)
-    (fp_text reference "R5" (at 3.556 0.508 90) (layer "B.SilkS")
+    (fp_text reference "R5" (at -1.92 0 180) (layer "B.SilkS")
       (effects (font (size 0.75 0.75) (thickness 0.15)) (justify mirror))
     )
@@
     (fp_line (start -1.98 -10.94) (end -3.18 -10.94) (layer "B.Fab") (width 0.1))
     (fp_line (start -3.18 4.1) (end -2.18 5.1) (layer "B.Fab") (width 0.1))
-    (pad "1" thru_hole roundrect (at 0 0 270) (size 1.7 1.7) (drill 1) (layers *.Cu *.Mask) (roundrect_rratio 0.147059)
+    (pad "1" thru_hole roundrect (at 0 0 270) (size 1.7 1.7) (drill 1) (layers *.Cu *.Mask) (roundrect_rratio 0.1470588235)
       (net 2 "/GATE1") (pinfunction "Pin_1") (pintype "passive"))
     (pad "2" thru_hole circle (at 2.54 0 270) (size 1.7 1.7) (drill 1) (layers *.Cu *.Mask)
@@
     (fp_line (start 3.81 2.92) (end -1.27 2.92) (layer "B.Fab") (width 0.1))
     (fp_line (start -1.27 0.5) (end -0.562893 0) (layer "B.Fab") (width 0.1))
-    (pad "1" thru_hole roundrect locked (at 0 0 270) (size 1.74 2.2) (drill 1.2) (layers *.Cu *.Mask) (roundrect_rratio 0.143678)
+    (pad "1" thru_hole roundrect locked (at 0 0 270) (size 1.74 2.2) (drill 1.2) (layers *.Cu *.Mask) (roundrect_rratio 0.1436781609)
       (net 20 "Net-(R9-Pad2)") (pinfunction "Pin_1") (pintype "passive"))
     (pad "2" thru_hole oval locked (at 2.54 0 270) (size 1.74 2.2) (drill 1.2) (layers *.Cu *.Mask)
@@
     (property "Vendor" "Tayda")
     (attr through_hole)
-    (fp_text reference "R6" (at 3.556 0.508 90) (layer "B.SilkS")
+    (fp_text reference "R6" (at -1.92 0 180) (layer "B.SilkS")
       (effects (font (size 0.75 0.75) (thickness 0.15)) (justify mirror))
     )
@@
     (property "Vendor" "Tayda")
     (attr through_hole)
-    (fp_text reference "R4" (at 3.556 0.508 90) (layer "B.SilkS")
+    (fp_text reference "R4" (at -1.92 0 180) (layer "B.SilkS")
       (effects (font (size 0.75 0.75) (thickness 0.15)) (justify mirror))
     )
@@
     (property "Vendor" "Tayda")
     (attr through_hole)
-    (fp_text reference "R7" (at 3.556 0.508 90) (layer "B.SilkS")
+    (fp_text reference "R7" (at -1.92 0 180) (layer "B.SilkS")
       (effects (font (size 0.75 0.75) (thickness 0.15)) (justify mirror))
     )
@@
     (property "Vendor" "Tayda")
     (attr through_hole)
-    (fp_text reference "R9" (at 3.556 0.508 90) (layer "B.SilkS")
+    (fp_text reference "R9" (at -1.92 -0.1 180) (layer "B.SilkS")
       (effects (font (size 0.75 0.75) (thickness 0.15)) (justify mirror))
     )
@@
     (property "Vendor" "Tayda")
     (attr through_hole)
-    (fp_text reference "R8" (at 3.556 0.508 90) (layer "B.SilkS")
+    (fp_text reference "R8" (at -1.92 -0.1 180) (layer "B.SilkS")
       (effects (font (size 0.75 0.75) (thickness 0.15)) (justify mirror))
     )
@@
     (property "Vendor" "Tayda")
     (attr through_hole)
-    (fp_text reference "R1" (at 3.556 0.508 90) (layer "B.SilkS")
-      (effects (font (size 0.75 0.75) (thickness 0.15)) (justify mirror))
-    )
+    (fp_text reference "R1" (at -1.82 0 180) (layer "B.SilkS")
+      (effects (font (size 0.75 0.75) (thickness 0.15)) (justify mirror))
+    )

Commit message: Minor Silkscreen Update
Parts:
- C1, C2: footprint ao_tht:C_Disc_D3.0mm_W1.6mm_P2.50mm -> ao_tht:C_Rect_L7.2mm_W2.5mm_P5.00mm_FKS2_FKP2_MKS2_MKP2
- moved C1 1.85 mm to (158.1, 107.0)
- moved C2 1.65 mm to (174.5, 107.1)
Routing:
- net Net-(R6-Pad2): track 41.5 -> 39.6 mm
- net /-12V: track 113.0 -> 113.9 mm
- net /+12V: track 81.0 -> 80.1 mm
