File: KosmoVoltsMain/KosmoVoltsMain.kicad_sch (KiCad schematic)
At the start: 22 parts, among them J1 OUT, J2 2_pin_Molex_connector, J3 OUT, U1 TL072

Commit message: Minor Silkscreen Update
Parts:
- C1, C2: footprint ao_tht:C_Disc_D3.0mm_W1.6mm_P2.50mm -> ao_tht:C_Rect_L7.2mm_W2.5mm_P5.00mm_FKS2_FKP2_MKS2_MKP2
Changed lines of the file:
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@@
       (effects (font (size 1.27 1.27)) (justify left))
     )
-    (property "Footprint" "ao_tht:C_Disc_D3.0mm_W1.6mm_P2.50mm" (id 2) (at 77.1652 181.61 0)
+    (property "Footprint" "ao_tht:C_Rect_L7.2mm_W2.5mm_P5.00mm_FKS2_FKP2_MKS2_MKP2" (id 2) (at 77.1652 181.61 0)
       (effects (font (size 1.27 1.27)) hide)
     )
@@
       (effects (font (size 1.27 1.27)) (justify left))
     )
-    (property "Footprint" "ao_tht:C_Disc_D3.0mm_W1.6mm_P2.50mm" (id 2) (at 77.1652 149.86 0)
+    (property "Footprint" "ao_tht:C_Rect_L7.2mm_W2.5mm_P5.00mm_FKS2_FKP2_MKS2_MKP2" (id 2) (at 77.1652 149.86 0)
       (effects (font (size 1.27 1.27)) hide)
     )
@@
     )
     (path "/af40b6da-1c42-4ccb-a147-e1d1e594c90c"
-      (reference "C1") (unit 1) (value "100n") (footprint "ao_tht:C_Disc_D3.0mm_W1.6mm_P2.50mm")
+      (reference "C1") (unit 1) (value "100n") (footprint "ao_tht:C_Rect_L7.2mm_W2.5mm_P5.00mm_FKS2_FKP2_MKS2_MKP2")
     )
     (path "/69582024-d92c-4de9-bbc9-8000c9b6c72d"
-      (reference "C2") (unit 1) (value "100n") (footprint "ao_tht:C_Disc_D3.0mm_W1.6mm_P2.50mm")
+      (reference "C2") (unit 1) (value "100n") (footprint "ao_tht:C_Rect_L7.2mm_W2.5mm_P5.00mm_FKS2_FKP2_MKS2_MKP2")
     )
     (path "/1cdc27ab-85a6-45f8-8c10-311802f8e75e"
